File: mcu-board/mcu board.kicad_pcb (KiCad board)
At the start: 4 copper layers, 92 x 82 mm, 35 parts, among them J1 USB_C, J2 Sensor_Forward, J3 Sensor_Right, J4 Sensor_Left, J5 I2C Breakout, J6 Conn_01x02, J7 Conn_01x02, J8 Conn_01x02, SW1 SW_SPST, SW2 SW_SPST, U1 ESP32-S3-1, U2 L7806, U3 L7806, U4 AZ1117-3.3

Commit message: implemented feedback
Parts:
- added R5: 150, Resistor_SMD:R_0603_1608Metric, F.Cu at (173.5, 107.0)
- added R6: 150, Resistor_SMD:R_0603_1608Metric, F.Cu at (120.0, 85.2)
Connections:
- net /MCU_IO15 renamed /FORWARD_INT
- net /MCU_IO16 renamed /RIGHT_INT
- net /MCU_IO17 renamed /LEFT_INT
- net /MCU_IO4 renamed /LEFT_SHUTDOWN
- net /MCU_IO6 renamed /FORWARD_SHUTDOWN
- net /MCU_IO7 renamed /RIGHT_SHUTDOWN
- D3 pad 1: GND -> Net-(D3-K)
- D4 pad 1: GND -> Net-(D4-K)
Routing:
- net +3.3V: track 203.6 -> 267.5 mm, vias 2 -> 3
- net Net-(D4-K): track 0.00 -> 4.01 mm
- net Net-(D3-K): track 0.00 -> 2.21 mm
- net GND: track 94.8 -> 95.8 mm
