File: mcu-board/mcu board.kicad_sch (KiCad schematic)
At the start: 17 parts, among them J1 USB_C, J2 Sensor_Forward, J3 Sensor_Right, J4 Sensor_Left, J5 I2C Breakout, SW1 SW_SPST, SW2 SW_SPST, U1 ESP32-S3-1

Commit message: implemented feedback
Parts:
- added R5: 150, Resistor_SMD:R_0603_1608Metric, symbol Device:R_Small_US
Connections:
- net GND: now also R5.1; no longer D4.1 (K)
- net MCU_IO15 renamed FORWARD_INT
- net MCU_IO16 renamed RIGHT_INT
- net MCU_IO17 renamed LEFT_INT
- net MCU_IO4 renamed LEFT_SHUTDOWN
- net MCU_IO6 renamed FORWARD_SHUTDOWN
- net MCU_IO7 renamed RIGHT_SHUTDOWN
- new net: D4.1 (K), R5.2
Changed lines of the file:
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@@
 	(text "blinky for testing mcu"
 		(exclude_from_sim no)
-		(at 217.932 47.244 0)
+		(at 212.09 43.942 0)
 		(effects
 			(font
@@
 	(wire
 		(pts
-			(xy 238.76 64.77) (xy 248.92 64.77)
+			(xy 228.6 64.77) (xy 248.92 64.77)
 		)
 		(stroke
@@
 	(wire
 		(pts
-			(xy 215.9 50.8) (xy 215.9 52.07)
+			(xy 151.13 31.75) (xy 151.13 33.02)
 		)
 		(stroke
@@
 	(wire
 		(pts
-			(xy 151.13 31.75) (xy 151.13 33.02)
+			(xy 234.95 33.02) (xy 248.92 33.02)
 		)
 		(stroke
@@
 	(wire
 		(pts
-			(xy 234.95 33.02) (xy 248.92 33.02)
+			(xy 114.3 55.88) (xy 116.84 55.88)
 		)
 		(stroke
@@
 	(wire
 		(pts
-			(xy 114.3 55.88) (xy 116.84 55.88)
+			(xy 215.9 50.8) (xy 215.9 53.34)
 		)
 		(stroke
@@
 	(wire
 		(pts
-			(xy 138.43 55.88) (xy 152.4 55.88)
+			(xy 133.35 55.88) (xy 152.4 55.88)
 		)
 		(stroke
@@
 	(wire
 		(pts
-			(xy 138.43 58.42) (xy 152.4 58.42)
+			(xy 133.35 58.42) (xy 152.4 58.42)
 		)
 		(stroke
@@
 	(wire
 		(pts
-			(xy 238.76 40.64) (xy 248.92 40.64)
+			(xy 236.22 40.64) (xy 248.92 40.64)
 		)
 		(stroke
@@
 	(wire
 		(pts
-			(xy 138.43 53.34) (xy 152.4 53.34)
+			(xy 133.35 53.34) (xy 152.4 53.34)
 		)
 		(stroke
@@
 	(wire
 		(pts
-			(xy 138.43 60.96) (xy 152.4 60.96)
+			(xy 133.35 60.96) (xy 152.4 60.96)
 		)
 		(stroke
@@
 	(wire
 		(pts
-			(xy 238.76 86.36) (xy 248.92 86.36)
+			(xy 228.6 86.36) (xy 248.92 86.36)
 		)
 		(stroke
@@
 	(wire
 		(pts
-			(xy 238.76 62.23) (xy 248.92 62.23)
+			(xy 237.49 62.23) (xy 248.92 62.23)
 		)
 		(stroke
@@
 	(wire
 		(pts
-			(xy 138.43 50.8) (xy 152.4 50.8)
+			(xy 133.35 50.8) (xy 152.4 50.8)
 		)
 		(stroke
@@
 	(wire
 		(pts
+			(xy 215.9 58.42) (xy 215.9 60.96)
+		)
+		(stroke
+			(width 0)
+			(type default)
+		)
+	)
+	(wire
+		(pts
 			(xy 119.38 36.83) (xy 114.3 36.83)
 		)
@@
 	(wire
 		(pts
-			(xy 238.76 83.82) (xy 248.92 83.82)
+			(xy 237.49 83.82) (xy 248.92 83.82)
 		)
 		(stroke
@@
 	(wire
 		(pts
-			(xy 238.76 43.18) (xy 248.92 43.18)
+			(xy 228.6 43.18) (xy 248.92 43.18)
 		)
 		(stroke
@@
 		)
 	)
-	(label "MCU_IO15"
-		(at 138.43 55.88 0)
+	(label "FORWARD_INT"
+		(at 133.35 55.88 0)
 		(effects
 			(font
@@
 		)
 	)
-	(label "MCU_IO4"
-		(at 238.76 86.36 0)
+	(label "LEFT_SHUTDOWN"
+		(at 228.6 86.36 0)
 		(effects
 			(font
@@
 		)
 	)
-	(label "MCU_IO16"
-		(at 138.43 58.42 0)
+	(label "RIGHT_INT"
+		(at 133.35 58.42 0)
 		(effects
 			(font
@@
 		)
 	)
-	(label "MCU_IO17"
-		(at 238.76 83.82 0)
+	(label "LEFT_INT"
+		(at 237.49 83.82 0)
 		(effects
 			(font
@@
 		)
 	)
-	(label "MCU_IO15"
-		(at 238.76 40.64 0)
+	(label "FORWARD_INT"
+		(at 236.22 40.64 0)
 		(effects
 			(font
@@
 		)
 	)
-	(label "MCU_IO17"
-		(at 138.43 60.96 0)
+	(label "LEFT_INT"
+		(at 133.35 60.96 0)
 		(effects
 			(font
@@
 		)
 	)
-	(label "MCU_IO6"
-		(at 138.43 50.8 0)
+	(label "FORWARD_SHUTDOWN"
+		(at 133.35 50.8 0)
 		(effects
 			(font
@@
 		)
 	)
-	(label "MCU_IO7"
-		(at 138.43 53.34 0)
+	(label "RIGHT_SHUTDOWN"
+		(at 133.35 53.34 0)
 		(effects
 			(font
@@
 		)
 	)
-	(label "MCU_IO4"
+	(label "LEFT_SHUTDOWN"
 		(at 138.43 45.72 0)
 		(effects
@@
 		)
 	)
-	(label "MCU_IO16"
-		(at 238.76 62.23 0)
+	(label "RIGHT_INT"
+		(at 237.49 62.23 0)
 		(effects
 			(font
@@
 		)
 	)
-	(label "MCU_IO6"
-		(at 238.76 43.18 0)
+	(label "FORWARD_SHUTDOWN"
+		(at 228.6 43.18 0)
 		(effects
 			(font
@@
 		)
 	)
-	(label "MCU_IO7"
-		(at 238.76 64.77 0)
+	(label "RIGHT_SHUTDOWN"
+		(at 228.6 64.77 0)
 		(effects
 			(font
@@
 		(on_board yes)
 		(dnp no)
-		(fields_autoplaced yes)
 		(property "Reference" "#PWR011"
 			(at 234.95 82.55 0)
@@
 		)
 		(property "Value" "GND"
-			(at 234.95 81.28 0)
+			(at 233.426 80.01 0)
 			(effects
 				(font
@@
 	(symbol
 		(lib_id "power:GND")
-		(at 215.9 52.07 0)
+		(at 215.9 60.96 0)
 		(mirror y)
 		(unit 1)
@@
 		(fields_autoplaced yes)
 		(property "Reference" "#PWR014"
-			(at 215.9 58.42 0)
+			(at 215.9 67.31 0)
 			(effects
 				(font
@@
 		)
 		(property "Value" "GND"
-			(at 215.9 57.15 0)
+			(at 215.9 66.04 0)
 			(effects
 				(font
@@
 		)
 		(property "Footprint" ""
-			(at 215.9 52.07 0)
+			(at 215.9 60.96 0)
 			(effects
 				(font
@@
 		)
 		(property "Datasheet" ""
-			(at 215.9 52.07 0)
+			(at 215.9 60.96 0)
 			(effects
 				(font
@@
 		)
 		(property "Description" "Power symbol creates a global label with name \"GND\" , ground"
-			(at 215.9 52.07 0)
+			(at 215.9 60.96 0)
 			(effects
 				(font
@@
 		(on_board yes)
 		(dnp no)
-		(fields_autoplaced yes)
 		(property "Reference" "#PWR012"
 			(at 234.95 60.96 0)
@@
 		)
 		(property "Value" "GND"
-			(at 234.95 59.69 0)
+			(at 233.426 58.928 0)
 			(effects
 				(font
@@
 		(on_board yes)
 		(dnp no)
-		(fields_autoplaced yes)
 		(property "Reference" "#PWR013"
 			(at 234.95 39.37 0)
@@
 		)
 		(property "Value" "GND"
-			(at 234.95 38.1 0)
+			(at 233.426 37.592 0)
 			(effects
 				(font
@@
 					(unit 1)
 				)
+			)
+		)
+	)
+	(symbol
+		(lib_id "Device:R_Small_US")
+		(at 215.9 55.88 180)
+		(unit 1)
+		(exclude_from_sim no)
+		(in_bom yes)
+		(on_board yes)
+		(dnp no)
+		(property "Reference" "R5"
+			(at 218.821 54.737 0)
+			(effects
+				(font
+					(size 1.27 1.27)
+				)
+			)
+		)
+		(property "Value" "150"
+			(at 219.456 56.388 0)
+			(effects
+				(font
+					(size 1.27 1.27)
+				)
+			)
+		)
+		(property "Footprint" "Resistor_SMD:R_0603_1608Metric"
+			(at 215.9 55.88 0)
+			(effects
+				(font
+					(size 1.27 1.27)
+				)
+				(hide yes)
+			)
+		)
+		(property "Datasheet" "~"
+			(at 215.9 55.88 0)
+			(effects
+				(font
+					(size 1.27 1.27)
+				)
+				(hide yes)
+			)
+		)
+		(property "Description" "Resistor, small US symbol"
+			(at 215.9 55.88 0)
+			(effects
+				(font
+					(size 1.27 1.27)
+				)
+				(hide yes)
+			)
+		)
+		(pin "1"
+		)
+		(pin "2"
+		)
+		(instances
+			(project "mcu board"
+				(path "/e926887c-cd26-4f47-be51-3352b14f6743"
+					(reference "R5")
+					(unit 1)
+				)
