File: mcu-board/power.kicad_sch (KiCad schematic)
At the start: 18 parts, among them J6 Conn_01x02, J7 Conn_01x02, J8 Conn_01x02, U2 L7806, U3 L7806, U4 AZ1117-3.3

Commit message: implemented feedback
Parts:
- added R6: 150, Resistor_SMD:R_0603_1608Metric, symbol Device:R_Small_US
Connections:
- net GND: now also R6.1; no longer D3.1 (K)
- new net: D3.1 (K), R6.2
Changed lines of the file:
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@@
+	(wire
+		(pts
+			(xy 31.75 154.94) (xy 31.75 157.48)
+		)
+		(stroke
+			(width 0)
+			(type default)
+		)
+	)
 	(wire
 		(pts
@@
 		(pts
 			(xy 228.6 87.63) (xy 219.71 87.63)
+		)
+		(stroke
+			(width 0)
+			(type default)
+		)
+	)
+	(wire
+		(pts
+			(xy 31.75 162.56) (xy 31.75 163.83)
 		)
 		(stroke
@@
 	(symbol
 		(lib_id "power:GND")
-		(at 31.75 154.94 0)
+		(at 31.75 163.83 0)
 		(unit 1)
 		(exclude_from_sim no)
@@
 		(fields_autoplaced yes)
 		(property "Reference" "#PWR04"
-			(at 31.75 161.29 0)
+			(at 31.75 170.18 0)
 			(effects
 				(font
@@
 		)
 		(property "Value" "GND"
-			(at 31.75 160.02 0)
+			(at 31.75 168.91 0)
 			(effects
 				(font
@@
 		)
 		(property "Footprint" ""
-			(at 31.75 154.94 0)
+			(at 31.75 163.83 0)
 			(effects
 				(font
@@
 		)
 		(property "Datasheet" ""
-			(at 31.75 154.94 0)
+			(at 31.75 163.83 0)
 			(effects
 				(font
@@
 		)
 		(property "Description" "Power symbol creates a global label with name \"GND\" , ground"
-			(at 31.75 154.94 0)
+			(at 31.75 163.83 0)
 			(effects
 				(font
@@
 					(unit 1)
 				)
+			)
+		)
+	)
+	(symbol
+		(lib_id "Device:R_Small_US")
+		(at 31.75 160.02 180)
+		(unit 1)
+		(exclude_from_sim no)
+		(in_bom yes)
+		(on_board yes)
+		(dnp no)
+		(property "Reference" "R6"
+			(at 34.671 158.877 0)
+			(effects
+				(font
+					(size 1.27 1.27)
+				)
+			)
+		)
+		(property "Value" "150"
+			(at 35.306 160.528 0)
+			(effects
+				(font
+					(size 1.27 1.27)
+				)
+			)
+		)
+		(property "Footprint" "Resistor_SMD:R_0603_1608Metric"
+			(at 31.75 160.02 0)
+			(effects
+				(font
+					(size 1.27 1.27)
+				)
+				(hide yes)
+			)
+		)
+		(property "Datasheet" "~"
+			(at 31.75 160.02 0)
+			(effects
+				(font
+					(size 1.27 1.27)
+				)
+				(hide yes)
+			)
+		)
+		(property "Description" "Resistor, small US symbol"
+			(at 31.75 160.02 0)
+			(effects
+				(font
+					(size 1.27 1.27)
+				)
+				(hide yes)
+			)
+		)
+		(pin "1"
+		)
+		(pin "2"
+		)
+		(instances
+			(project "mcu board"
+				(path "/e926887c-cd26-4f47-be51-3352b14f6743/65b6e221-2db7-4e52-96fb-70ae76f49758"
+					(reference "R6")
+					(unit 1)
+				)
